File: PCB/DangerDoughnut/DangerDoughnut.kicad_pcb (KiCad board)
At the start: 4 copper layers, 50 x 37 mm, 157 parts, among them J1 Conn_01x02_Pin, J10 Conn_01x01_Pin, J11 Conn_01x01_Pin, J12 Conn_01x01_Pin, J13 Conn_01x01_Pin, J14 Conn_01x01_Pin, J15 Conn_01x01_Pin, J16 Conn_01x01_Pin, J17 Conn_01x01_Pin, J19 Conn_01x01_Pin, J2 Conn_01x02_Pin, J20 Conn_01x01_Pin, J3 Conn_01x02_Pin, J4 Conn_01x04_Pin, J6 USB_C_Receptacle_USB2.0_16P, J7 Conn_01x01_Pin, J8 Conn_01x01_Pin, J9 Conn_01x01_Pin, SW1 SW_Push, SW2 SW_Push, U1 MMC5983MA, U10 ESP32-S3, U2 H3LIS331DLTR, U3 H3LIS331DLTR, U4 W25X20CLZP, U6 L5973D, U7 MIC5219-3.3YM5, U8 ESP8285H16, U9 SX1280IMLTRT, Y1 40MHz, Y2 52MHz, Y3 26MHz

Commit message: Layout Done
Parts:
- added C43: 20pF, Capacitor_SMD:C_0402_1005Metric_Pad0.74x0.62mm_HandSolder, F.Cu at (87.1, 70.6)
- added C44: 20pF, Capacitor_SMD:C_0402_1005Metric_Pad0.74x0.62mm_HandSolder, F.Cu at (90.9, 70.5)
- moved TP20 1.90 mm to (88.2, 43.0)
- moved TP8 0.95 mm to (91.1, 68.3)
- moved C22 0.40 mm to (86.1, 70.5)
- moved C16 0.40 mm to (84.9, 70.4)
Connections:
- J11 pad 1: Net-(J11-Pin_1) -> GND
- U10 pad 24: Net-(J11-Pin_1) -> unconnected-(U10-GPIO18-Pad24)
Routing:
- net Net-(J11-Pin_1): track 34.3 -> 0.00 mm, vias 4 -> 0
- net +3.3V: track 87.1 -> 110.6 mm, vias 36 -> 41
- net Net-(U9-XTB): track 2.13 -> 3.33 mm
- net BATT: track 39.2 -> 38.1 mm
- net Net-(D2-A): track 22.5 -> 21.5 mm
- net ELSR_TX: track 21.1 -> 22.2 mm
- net Net-(U9-XTA): track 3.26 -> 4.23 mm
- net /DCC_FB: track 10.7 -> 11.2 mm
- net ESC_L: track 17.1 -> 17.7 mm
- net Net-(J8-Pin_1): track 39.1 -> 38.6 mm
- net GND: vias 175 -> 298

Commit message: boards ordered
Parts:
- added ?: , , F.Cu at (87.6, 78.1)
- added ?: , , F.Cu at (92.8, 78.8)
- added ?: , , F.Cu at (94.2, 79.6)
- added ?: , , F.Cu at (86.3, 78.1)
- added ?: , , F.Cu at (90.2, 79.6)
- added ?: , , F.Cu at (103.2, 79.6)
- added ?: , , F.Cu at (121.4, 78.8)
- added ?: , , F.Cu at (102.0, 78.8)
- added ?: , , F.Cu at (74.6, 78.8)
- added ?: , , F.Cu at (104.5, 78.8)
- added ?: , , F.Cu at (115.0, 78.1)
- added ?: , , F.Cu at (107.2, 78.1)
- added ?: , , F.Cu at (96.8, 78.1)
- added ?: , , F.Cu at (104.5, 79.6)
- added ?: , , F.Cu at (78.5, 78.8)
- added ?: , , F.Cu at (77.2, 78.1)
- added ?: , , F.Cu at (120.2, 78.1)
- added ?: , , F.Cu at (89.0, 79.6)
- added ?: , , F.Cu at (81.2, 79.6)
- added ?: , , F.Cu at (77.2, 78.8)
- added ?: , , F.Cu at (96.8, 79.6)
- added ?: , , F.Cu at (90.2, 78.8)
- added ?: , , F.Cu at (103.2, 78.8)
- added ?: , , F.Cu at (98.0, 79.6)
- added ?: , , F.Cu at (78.5, 78.1)
- added ?: , , F.Cu at (116.2, 78.8)
- added ?: , , F.Cu at (124.0, 79.6)
- added ?: , , F.Cu at (79.8, 78.1)
- added ?: , , F.Cu at (109.8, 78.8)
- added ?: , , F.Cu at (83.8, 78.1)
- added ?: , , F.Cu at (94.2, 78.1)
- added ?: , , F.Cu at (95.4, 78.8)
- added ?: , , F.Cu at (85.0, 79.6)
- added ?: , , F.Cu at (91.5, 78.1)
- added ?: , , F.Cu at (117.5, 78.8)
- added ?: , , F.Cu at (102.0, 79.6)
- added ?: , , F.Cu at (82.4, 78.1)
- added ?: , , F.Cu at (92.8, 78.1)
- added ?: , , F.Cu at (105.8, 78.1)
- added ?: , , F.Cu at (87.6, 79.6)
- added ?: , , F.Cu at (95.4, 78.1)
- added ?: , , F.Cu at (96.8, 78.8)
- added ?: , , F.Cu at (102.0, 78.1)
- added ?: , , F.Cu at (74.6, 78.1)
- added ?: , , F.Cu at (79.8, 78.8)
- added ?: , , F.Cu at (112.3, 78.8)
- added ?: , , F.Cu at (83.8, 78.8)
- added ?: , , F.Cu at (76.0, 79.6)
- added ?: , , F.Cu at (122.8, 78.1)
- added ?: , , F.Cu at (100.6, 79.6)
- added ?: , , F.Cu at (82.4, 78.8)
- added ?: , , F.Cu at (118.8, 78.8)
- added ?: , , F.Cu at (83.8, 79.6)
- added ?: , , F.Cu at (99.3, 79.6)
- added ?: , , F.Cu at (117.5, 79.6)
- added ?: , , F.Cu at (108.4, 78.1)
- added ?: , , F.Cu at (90.2, 78.1)
- added ?: , , F.Cu at (120.2, 79.6)
- added ?: , , F.Cu at (121.4, 79.6)
- added ?: , , F.Cu at (122.8, 78.8)
- added ?: , , F.Cu at (113.6, 79.6)
- added ?: , , F.Cu at (120.2, 78.8)
- added ?: , , F.Cu at (107.2, 78.8)
- added ?: , , F.Cu at (117.5, 78.1)
- added ?: , , F.Cu at (111.0, 78.1)
- added ?: , , F.Cu at (89.0, 78.1)
- added ?: , , F.Cu at (91.5, 78.8)
- added ?: , , F.Cu at (109.8, 78.1)
- added ?: , , F.Cu at (85.0, 78.1)
- added ?: , , F.Cu at (86.3, 78.8)
- added ?: , , F.Cu at (104.5, 78.1)
- added ?: , , F.Cu at (94.2, 78.8)
- added ?: , , F.Cu at (109.8, 79.6)
- added ?: , , F.Cu at (86.3, 79.6)
- added ?: , , F.Cu at (82.4, 79.6)
- added ?: , , F.Cu at (92.8, 79.6)
- added ?: , , F.Cu at (113.6, 78.1)
- added ?: , , F.Cu at (116.2, 78.1)
- added ?: , , F.Cu at (81.2, 78.8)
- added ?: , , F.Cu at (118.8, 79.6)
- added ?: , , F.Cu at (113.6, 78.8)
- added ?: , , F.Cu at (108.4, 78.8)
- added ?: , , F.Cu at (111.0, 78.8)
- added ?: , , F.Cu at (89.0, 78.8)
- added ?: , , F.Cu at (124.0, 78.1)
- added ?: , , F.Cu at (125.3, 79.6)
- added ?: , , F.Cu at (95.4, 79.6)
- added ?: , , F.Cu at (76.0, 78.1)
- added ?: , , F.Cu at (107.2, 79.6)
- added ?: , , F.Cu at (111.0, 79.6)
- added ?: , , F.Cu at (91.5, 79.6)
- added ?: , , F.Cu at (112.3, 78.1)
- added ?: , , F.Cu at (124.0, 78.8)
- added ?: , , F.Cu at (81.2, 78.1)
- added ?: , , F.Cu at (115.0, 78.8)
- added ?: , , F.Cu at (74.6, 79.6)
- added ?: , , F.Cu at (116.2, 79.6)
- added ?: , , F.Cu at (103.2, 78.1)
- added ?: , , F.Cu at (98.0, 78.8)
- added ?: , , F.Cu at (78.5, 79.6)
- added ?: , , F.Cu at (100.6, 78.8)
- added ?: , , F.Cu at (105.8, 79.6)
- added ?: , , F.Cu at (125.3, 78.1)
- added ?: , , F.Cu at (122.8, 79.6)
- added ?: , , F.Cu at (100.6, 78.1)
- added ?: , , F.Cu at (87.6, 78.8)
- added ?: , , F.Cu at (112.3, 79.6)
- added ?: , , F.Cu at (105.8, 78.8)
- added ?: , , F.Cu at (118.8, 78.1)
- added ?: , , F.Cu at (121.4, 78.1)
- added ?: , , F.Cu at (76.0, 78.8)
- added ?: , , F.Cu at (79.8, 79.6)
- added ?: , , F.Cu at (85.0, 78.8)
- added ?: , , F.Cu at (125.3, 78.8)
- added ?: , , F.Cu at (115.0, 79.6)
- added ?: , , F.Cu at (108.4, 79.6)
- added ?: , , F.Cu at (99.3, 78.1)
- added ?: , , F.Cu at (98.0, 78.1)
- added ?: , , F.Cu at (99.3, 78.8)
- added ?: , , F.Cu at (77.2, 79.6)
- added TP29: GND, Danger_Doughnut_Lib:Test_Via, F.Cu at (108.0, 49.0)
- added TP30: GND, Danger_Doughnut_Lib:Test_Via, F.Cu at (79.8, 42.8)
- C41: footprint Capacitor_SMD:C_0603_1608Metric -> Capacitor_SMD:C_0402_1005Metric
- J1: value Conn_01x02_Pin -> Battery
- J2: value Conn_01x02_Pin -> ESC_R
- J3: value Conn_01x02_Pin -> ESC_L
- J4: value Conn_01x04_Pin -> LED_Strip
- moved TP23 11.7 mm to (96.5, 61.5)
- moved TP4 11.0 mm to (98.2, 62.2)
- moved TP17 10.8 mm to (97.2, 62.0)
Connections:
- net Net-(U9-RFIO) renamed SX_Ant
Routing:
- net +3.3V: track 110.6 -> 111.1 mm
- net GND: vias 298 -> 295

Commit message: added a few things
Parts:
- removed kibuzzard-668D7854: G***, kibuzzard-668D7854
- added kibuzzard-672AA985: G***, kibuzzard-672AA985, F.Cu at (106.0, 61.0)
