File: PCB/DangerDoughnut/DangerDoughnut.kicad_sch (KiCad schematic)
At the start: 154 parts, among them J1 Conn_01x02_Pin, J10 Conn_01x01_Pin, J11 Conn_01x01_Pin, J12 Conn_01x01_Pin, J13 Conn_01x01_Pin, J14 Conn_01x01_Pin, J15 Conn_01x01_Pin, J16 Conn_01x01_Pin, J17 Conn_01x01_Pin, J19 Conn_01x01_Pin, J2 Conn_01x02_Pin, J20 Conn_01x01_Pin, J3 Conn_01x02_Pin, J4 Conn_01x04_Pin, J6 USB_C_Receptacle_USB2.0_16P, J7 Conn_01x01_Pin, J8 Conn_01x01_Pin, J9 Conn_01x01_Pin, SW1 SW_Push, SW2 SW_Push, U1 MMC5983MA, U10 ESP32-S3, U2 H3LIS331DLTR, U3 H3LIS331DLTR, U4 W25X20CLZP, U6 L5973D, U7 MIC5219-3.3YM5, U8 ESP8285H16, U9 SX1280IMLTRT, Y1 40MHz, Y2 52MHz, Y3 26MHz

Commit message: boards ordered
Parts:
- added TP29, TP30: GND, Danger_Doughnut_Lib:Test_Via, symbol Connector:TestPoint
- C41: footprint Capacitor_SMD:C_0603_1608Metric -> Capacitor_SMD:C_0402_1005Metric
- J1: value Conn_01x02_Pin -> Battery
- J2: value Conn_01x02_Pin -> ESC_R
- J3: value Conn_01x02_Pin -> ESC_L
- J4: value Conn_01x04_Pin -> LED_Strip
Connections:
- net GND: now also TP29.1, TP30.1
- net SX_Ant: now reaches FL1.1, U9.22 (RFIO)
Other:
- note added: "ESP32-S3"
- note added: "LEDs/ESC"
- note added: "Power Supply"
- note added: "Radio"
- note added: "Sensors"
- note added: "Test Points"
- note added: "USB"
- note removed: "TODO: Organize"
- moved on the sheet: ANT1, ANT2, C1, C10, C11, C12, C13, C14, C15, C16, C17, C18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

Commit message: update
Other:
- note added: "TODO: flat antenna"
- note added: "TODO: reset button"
